Commit message: 仿真里面已经初步完成稳定站立

File: src/model/model/wheel_leg.urdf (robot description, URDF)
Before this commit: robot wheel_leg, 8 links, 7 joints
Links:
- removed link imu_link
- removed link leg_left_shank
- removed link leg_left_thigh
- removed link leg_right_shank
- removed link leg_right_thigh
- removed link wheel_left
- removed link wheel_right
- added link lb_link1, mass 0.0157407698288876; collision mesh filename=package://model/meshes/lb_link1.STL; visual mesh filename=package://model/meshes/lb_link1.STL
- added link lb_link2, mass 0.0441319313931042; collision mesh filename=package://model/meshes/lb_link2.STL; visual mesh filename=package://model/meshes/lb_link2.STL
- added link lefoot_link, mass 0.130114342543911; collision mesh filename=package://model/meshes/lefoot_link.STL; visual mesh filename=package://model/meshes/lefoot_link.STL
- added link lf_link1, mass 0.0228632381715483; collision mesh filename=package://model/meshes/lf_link1.STL; visual mesh filename=package://model/meshes/lf_link1.STL
- added link lf_link2, mass 0.0355326730325909; collision mesh filename=package://model/meshes/lf_link2.STL; visual mesh filename=package://model/meshes/lf_link2.STL
- added link rb_link1, mass 0.0157407698288876; collision mesh filename=package://model/meshes/rb_link1.STL; visual mesh filename=package://model/meshes/rb_link1.STL
- added link rb_link2, mass 0.0441319313931042; collision mesh filename=package://model/meshes/rb_link2.STL; visual mesh filename=package://model/meshes/rb_link2.STL
- added link rf_link1, mass 0.0228632381715483; collision mesh filename=package://model/meshes/rf_link1.STL; visual mesh filename=package://model/meshes/rf_link1.STL
- added link rf_link2, mass 0.0355326730325909; collision mesh filename=package://model/meshes/rf_link2.STL; visual mesh filename=package://model/meshes/rf_link2.STL
- added link rifoot_link, mass 0.15505019042519; collision mesh filename=package://model/meshes/rifoot_link.STL; visual mesh filename=package://model/meshes/rifoot_link.STL
- link base_link: mass 1.0 -> 1.66745151375332; geometry collision mesh filename=package://model/meshes/base_link.STL; visual mesh filename=package://model/meshes/base_link.STL
Joints:
- removed joint imu_joint
- removed joint leg_left_hip_joint
- removed joint leg_left_knee_joint
- removed joint leg_right_hip_joint
- removed joint leg_right_knee_joint
- removed joint wheel_left_joint
- removed joint wheel_right_joint
- added joint lb_joint1: type revolute, parent base_link, child lb_link1, origin xyz=-0.030794 0.125500 0.149300 rpy=-1.5708 0 0, axis 0 0 -1, limit lower=-2.0 upper=2.0 effort=12.0 velocity=20.0
- added joint lb_joint2: type revolute, parent lb_link1, child lb_link2, origin xyz=-0.041299 0.028185 0.01 rpy=0 0 2.5427, axis 0 0 -1, limit lower=-3.1416 upper=3.1416 effort=1.0 velocity=20.0
- added joint lefoot_joint: type continuous, parent lf_link2, child lefoot_link, origin xyz=0.022658 0.10253 0.0215 rpy=0 0 1.3533, axis 0 0 -1, limit effort=3.0 velocity=40.0
- added joint lf_joint1: type revolute, parent base_link, child lf_link1, origin xyz=0.029206 0.131000 0.149300 rpy=-1.5708 0 0, axis 0 0 -1, limit lower=-2.0 upper=2.0 effort=12.0 velocity=20.0
- added joint lf_joint2: type revolute, parent lf_link1, child lf_link2, origin xyz=0.0275573394802777 0.0417204151557571 0 rpy=0 0 0.987058337135097, axis 0 0 -1, limit lower=-3.1416 upper=3.1416 effort=1.0 velocity=20.0
- added joint rb_joint1: type revolute, parent base_link, child rb_link1, origin xyz=-0.030794 -0.125496 0.149300 rpy=1.5708 0 0, axis 0 0 -1, limit lower=-2.0 upper=2.0 effort=12.0 velocity=20.0
- added joint rb_joint2: type revolute, parent rb_link1, child rb_link2, origin xyz=-0.028236 -0.041264 0 rpy=0 0 -2.1709, axis 0 0 -1, limit lower=-3.1416 upper=3.1416 effort=1.0 velocity=20.0
- added joint rf_joint1: type revolute, parent base_link, child rf_link1, origin xyz=0.029206 -0.131000 0.149300 rpy=1.5708 0 0, axis 0 0 -1, limit lower=-2.0 upper=2.0 effort=12.0 velocity=20.0
- added joint rf_joint2: type revolute, parent rf_link1, child rf_link2, origin xyz=0.0249005076512295 -0.0433585599243225 0 rpy=0 0 -1.04949370860079, axis 0 0 -1, limit lower=-3.1416 upper=3.1416 effort=1.0 velocity=20.0
- added joint rifoot_joint: type continuous, parent rf_link2, child rifoot_link, origin xyz=0.046796 -0.093996 0.0215 rpy=0 0 -1.1089, axis 0 0 -1, limit effort=3.0 velocity=40.0
